File: CANopus/ECU_ADC.kicad_sch (KiCad schematic)
At the start: 1 part

Commit message: Analog modifs
Signed-off-by: mat7784 <matispoulin@gmail.com>
Parts:
- added U4: INA826, UserFootprints:SOP65P490X110-8N, symbol INA826:INA826AIDGKR
Connections:
- net Pressure Sensor 1: now reaches D3.1 (K)
- net Pressure Sensor 1: now also U4.7 (Vout)
Other:
- note added: "PT Chambre"
- moved on the sheet: D3
Changed lines of the file:
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@@
 	(rectangle
 		(start 30.48 27.94)
-		(end 139.7 101.6)
+		(end 113.03 101.6)
 		(stroke
 			(width 0)
@@
 		)
 	)
+	(text "PT Chambre"
+		(exclude_from_sim no)
+		(at 37.846 30.734 0)
+		(effects
+			(font
+				(size 1.27 1.27)
+			)
+		)
+	)
+	(junction
+		(at 92.71 53.34)
+		(diameter 0)
+		(color 0 0 0 0)
+	)
 	(wire
 		(pts
-			(xy 59.69 80.01) (xy 59.69 83.82)
+			(xy 74.93 53.34) (xy 92.71 53.34)
 		)
 		(stroke
@@
 		)
 	)
+	(wire
+		(pts
+			(xy 92.71 53.34) (xy 97.79 53.34)
+		)
+		(stroke
+			(width 0)
+			(type default)
+		)
+	)
+	(wire
+		(pts
+			(xy 92.71 63.5) (xy 92.71 67.31)
+		)
+		(stroke
+			(width 0)
+			(type default)
+		)
+	)
+	(label "Pressure Sensor 1"
+		(at 97.79 53.34 0)
+		(effects
+			(font
+				(size 1.27 1.27)
+			)
+			(justify left bottom)
+		)
+	)
 	(symbol
 		(lib_id "power:GND")
-		(at 59.69 83.82 0)
+		(at 92.71 67.31 0)
 		(unit 1)
 		(exclude_from_sim no)
@@
 		(fields_autoplaced yes)
 		(property "Reference" "#PWR053"
-			(at 59.69 90.17 0)
+			(at 92.71 73.66 0)
 			(effects
 				(font
@@
 		)
 		(property "Value" "GND"
-			(at 59.69 88.9 0)
+			(at 92.71 72.39 0)
 			(effects
 				(font
@@
 		)
 		(property "Footprint" ""
-			(at 59.69 83.82 0)
+			(at 92.71 67.31 0)
 			(effects
 				(font
@@
 		)
 		(property "Datasheet" ""
-			(at 59.69 83.82 0)
+			(at 92.71 67.31 0)
 			(effects
 				(font
@@
 		)
 		(property "Description" "Power symbol creates a global label with name \"GND\" , ground"
-			(at 59.69 83.82 0)
+			(at 92.71 67.31 0)
 			(effects
 				(font
@@
 	(symbol
 		(lib_id "0CSL_D1_V1:DIODE_SCHOTTKY_30V_200mA")
-		(at 59.69 74.93 270)
+		(at 92.71 58.42 270)
 		(unit 1)
 		(exclude_from_sim no)
@@
 		(fields_autoplaced yes)
 		(property "Reference" "D3"
-			(at 62.23 73.3424 90)
+			(at 95.25 56.8324 90)
 			(effects
 				(font
@@
 		)
 		(property "Value" "6.4V"
-			(at 62.23 75.8824 90)
+			(at 95.25 59.3724 90)
 			(effects
 				(font
@@
 		)
 		(property "Footprint" "Diode_SMD:D_0603_1608Metric_Pad1.05x0.95mm_HandSolder"
-			(at 55.245 74.93 0)
+			(at 88.265 58.42 0)
 			(effects
 				(font
@@
 		)
 		(property "Datasheet" ""
-			(at 59.69 74.93 0)
+			(at 92.71 58.42 0)
 			(effects
 				(font
@@
 		)
 		(property "Description" "Diode Schottky 30V 200mA (DC) Surface Mount SOD-123"
-			(at 59.69 74.93 0)
+			(at 92.71 58.42 0)
 			(effects
 				(font
@@
 		)
 		(property "Part Number" "1727-7327-1-ND"
-			(at 59.69 74.93 0)
+			(at 92.71 58.42 0)
 			(effects
 				(font
@@
 		)
 		(property "Link" "https://www.digikey.ca/en/products/detail/texas-instruments/INA826AIDGKR/2762216"
-			(at 59.69 74.93 0)
+			(at 92.71 58.42 0)
 			(effects
 				(font
@@
 	(symbol
 		(lib_id "power:VDD")
-		(at 39.37 50.8 0)
+		(at 44.45 45.72 0)
 		(unit 1)
 		(exclude_from_sim no)
@@
 		(dnp no)
 		(property "Reference" "#PWR052"
-			(at 39.37 54.61 0)
+			(at 44.45 49.53 0)
 			(effects
 				(font
@@
 		)
 		(property "Value" "VDDA"
-			(at 39.37 45.085 90)
+			(at 44.45 40.005 90)
 			(effects
 				(font
@@
 		)
 		(property "Footprint" ""
-			(at 39.37 50.8 0)
+			(at 44.45 45.72 0)
 			(effects
 				(font
@@
 		)
 		(property "Datasheet" ""
-			(at 39.37 50.8 0)
+			(at 44.45 45.72 0)
 			(effects
 				(font
@@
 		)
 		(property "Description" "Power symbol creates a global label with name \"VDD\""
-			(at 39.37 50.8 0)
+			(at 44.45 45.72 0)
 			(effects
 				(font
@@
 					(unit 1)
 				)
+			)
+		)
+	)
+	(symbol
+		(lib_id "INA826:INA826AIDGKR")
+		(at 64.77 53.34 0)
+		(unit 1)
+		(exclude_from_sim no)
+		(in_bom yes)
+		(on_board yes)
+		(dnp no)
+		(property "Reference" "U4"
+			(at 69.85 49.53 0)
+			(effects
+				(font
+					(size 1.27 1.27)
+				)
+			)
+		)
+		(property "Value" "INA826"
+			(at 71.755 56.515 0)
+			(effects
+				(font
+					(size 1.27 1.27)
+				)
+			)
+		)
+		(property "Footprint" "UserFootprints:SOP65P490X110-8N"
+			(at 64.77 53.34 0)
+			(effects
+				(font
+					(size 1.27 1.27)
+				)
+				(justify bottom)
+				(hide yes)
+			)
+		)
+		(property "Datasheet" ""
+			(at 64.77 53.34 0)
+			(effects
+				(font
+					(size 1.27 1.27)
+				)
+				(hide yes)
+			)
+		)
+		(property "Description" ""
+			(at 64.77 53.34 0)
+			(effects
+				(font
+					(size 1.27 1.27)
+				)
+				(hide yes)
+			)
+		)
+		(property "PARTREV" "G"
+			(at 64.77 53.34 0)
+			(effects
+				(font
+					(size 1.27 1.27)
+				)
+				(justify bottom)
+				(hide yes)
+			)
+		)
+		(property "STANDARD" "IPC-7351B"
+			(at 64.77 53.34 0)
+			(effects
+				(font
+					(size 1.27 1.27)
+				)
+				(justify bottom)
+				(hide yes)
+			)
+		)
+		(property "MAXIMUM_PACKAGE_HEIGHT" "1.10 mm"
+			(at 64.77 53.34 0)
+			(effects
+				(font
+					(size 1.27 1.27)
+				)
+				(justify bottom)
+				(hide yes)
+			)
+		)
+		(property "MANUFACTURER" "Texas Instruments"
+			(at 64.77 53.34 0)
+			(effects
+				(font
+					(size 1.27 1.27)
+				)
+				(justify bottom)
+				(hide yes)
+			)
+		)
+		(property "Digikey" ""
+			(at 64.77 53.34 0)
+			(effects
+				(font
+					(size 1.27 1.27)
+				)
+				(hide yes)
+			)
+		)
+		(property "Part Number" ""
+			(at 64.77 53.34 0)
+			(effects
+				(font
+					(size 1.27 1.27)
+				)
+				(hide yes)
+			)
+		)
+		(pin "5"
+		)
+		(pin "3"
+		)
+		(pin "6"
+		)
+		(pin "1"
+		)
+		(pin "2"
+		)
+		(pin "4"
+		)
+		(pin "8"
+		)
+		(pin "7"
+		)
+		(instances
+			(project "CANopus"
+				(path "/dca285e3-1f01-49ba-8aea-086d886ed352/6241f3be-b688-414f-b6ea-3b2705385d94"
+					(reference "U4")
+					(unit 1)
+				)
