File: CANopus/CANopus.kicad_pcb (KiCad board)
At the start: 2 copper layers, 3 parts, among them J1 Micro_SD_Card_Det1, J2 Micro_SD_Card_Det1, U2 STM32H747IITx

Commit message: Pages cleanup
Parts:
- added BZ1: Buzzer_TDK_PS1240, 0CSL_D1_V1:Buzzer_TDK_PS1240P02BT_D12.2mmP5mm, F.Cu at (64.2, 45.8)
- added C34: 0.1u, Capacitor_SMD:C_0603_1608Metric_Pad1.08x0.95mm_HandSolder, F.Cu at (67.1, 73.5)
- added C35: 0.1uF, Capacitor_SMD:C_0603_1608Metric_Pad1.08x0.95mm_HandSolder, F.Cu at (67.1, 76.0)
- added C36: 0.47uF, Capacitor_SMD:C_0603_1608Metric_Pad1.08x0.95mm_HandSolder, F.Cu at (67.1, 78.5)
- added C38: 0.1uF, Capacitor_SMD:C_0603_1608Metric_Pad1.08x0.95mm_HandSolder, F.Cu at (67.1, 81.0)
- added C39: 10uF/50V, Capacitor_SMD:CP_Elec_4x5.4, F.Cu at (77.5, 41.9)
- added D1: D, Diode_SMD:D_0603_1608Metric_Pad1.05x0.95mm_HandSolder, F.Cu at (75.8, 46.1)
- added D2: 6.4V, Diode_SMD:D_0603_1608Metric_Pad1.05x0.95mm_HandSolder, F.Cu at (75.8, 48.7)
- added D3: 6.4V, Diode_SMD:D_0603_1608Metric_Pad1.05x0.95mm_HandSolder, F.Cu at (76.9, 86.5)
- added F1: Polyfuse, Fuse:Fuse_0603_1608Metric_Pad1.05x0.95mm_HandSolder, F.Cu at (67.1, 83.5)
- added J17: USB_C_Receptacle_USB2.0_man, Connector_USB:USB_C_Receptacle_GCT_USB4105-xx-A_16P_TopMnt_Horizontal, F.Cu at (73.0, 97.5)
- added R27: 5.1k, Resistor_SMD:R_0603_1608Metric_Pad0.98x0.95mm_HandSolder, F.Cu at (67.1, 86.0)
- added R28: 5.1k, Resistor_SMD:R_0603_1608Metric_Pad0.98x0.95mm_HandSolder, F.Cu at (67.1, 88.6)
- added U1: SST25VF080B-50-4x-S2Ax, Package_SO:SOIC-8_5.3x5.3mm_P1.27mm, F.Cu at (43.0, 62.0)
- added U9: USBLC6-2SC6, Package_TO_SOT_SMD:SOT-23-6, F.Cu at (73.9, 62.0)
Connections:
- net Net-(U2-VDD33_USB) renamed VDD33_USB
- net Net-(U2-VDD50_USB) renamed VDD50_USB
- J1 pad 1: unconnected-(J1-DAT2-Pad1) -> /DAT2_SD1
- J1 pad 10: unconnected-(J1-SHIELD-Pad10) -> GND
- J1 pad 2: unconnected-(J1-DAT3/CD-Pad2) -> /DAT3_SD1
- J1 pad 3: unconnected-(J1-CMD-Pad3) -> /CMD_SD1
- J1 pad 4: unconnected-(J1-VDD-Pad4) -> +3V3
- J1 pad 5: unconnected-(J1-CLK-Pad5) -> /CLK_SD1
- J1 pad 6: unconnected-(J1-VSS-Pad6) -> GND
- J1 pad 7: unconnected-(J1-DAT0-Pad7) -> /DAT0_SD1
- J1 pad 8: unconnected-(J1-DAT1-Pad8) -> /DAT1_SD1
- J1 pad 9: unconnected-(J1-DET-Pad9) -> /DET_SD1
- U2 pad 101: unconnected-(U2-VCAPDSI-Pad101) -> VCAPDSI
- U2 pad 135: VCAP -> VDDLDO
- U2 pad 167: unconnected-(U2-BOOT0-Pad167) -> /BOOT0
- U2 pad 17: VCAP -> /VFBSMPS
- U2 pad 175: VCAP -> VDDLDO
- U2 pad 33: unconnected-(U2-NRST-Pad33) -> /NRST
- U2 pad 39: unconnected-(U2-VREF+-Pad39) -> VREF
- U2 pad 82: VCAP -> VDDLDO

Commit message: library
Signed-off-by: mat7784 <matispoulin@gmail.com>
Parts:
- turned U2 to -90 degrees

Commit message: Alim
Parts:
- removed J1, J2: Micro_SD_Card_Det1, UserFootprints:GCT_MEM2075-00-140-01-A
- added BT1: Battery_Holder_1025, 0CSL_D1_V1:BatteryHolder_BHX1_1025, F.Cu at (65.5, 95.8)
- added C45: 10u, 0CSL_D1_V1:C0805_MAN, F.Cu at (67.0, 43.0)
- added C46: 10u, 0CSL_D1_V1:C0805_MAN, F.Cu at (67.0, 46.2)
- added C47: 10u, 0CSL_D1_V1:C0603_MAN, F.Cu at (71.6, 47.0)
- added C48: 100n, 0CSL_D1_V1:C0603_MAN, F.Cu at (71.6, 49.7)
- added C49: 10u, 0CSL_D1_V1:C0603_MAN, F.Cu at (71.6, 52.4)
- added C50: 22u, 0CSL_D1_V1:C0805_MAN, F.Cu at (67.0, 49.5)
- added C51: 22u, 0CSL_D1_V1:C0805_MAN, F.Cu at (67.0, 52.8)
- added C52: 22u, 0CSL_D1_V1:C0805_MAN, F.Cu at (61.5, 50.0)
- added C53: 4.7u, 0CSL_D1_V1:C0805_MAN, F.Cu at (98.4, 27.0)
- added C54: 4.7u, 0CSL_D1_V1:C0805_MAN, F.Cu at (98.4, 30.3)
- added C55: 100n, 0CSL_D1_V1:C0603_MAN, F.Cu at (105.4, 33.9)
- added C56: 390pF, 0CSL_D1_V1:C0805_MAN, F.Cu at (98.4, 33.5)
- added C57: 10pF, 0CSL_D1_V1:C0805_MAN, F.Cu at (98.4, 36.8)
- added C58: 22uF, 0CSL_D1_V1:C0805_MAN, F.Cu at (98.4, 40.0)
- added R10: 100k, 0CSL_D1_V1:R0603_MAN, F.Cu at (61.5, 60.0)
- added R11: 150k, 0CSL_D1_V1:R0603_MAN, F.Cu at (70.9, 56.0)
- added R2: 10k, Resistor_SMD:R_0603_1608Metric_Pad0.98x0.95mm_HandSolder, F.Cu at (80.9, 87.5)
- added R3: 57.6k, 0CSL_D1_V1:R0603_MAN, F.Cu at (105.4, 26.1)
- added R4: x, 0CSL_D1_V1:R0603_MAN, F.Cu at (105.4, 28.8)
- added R5: x, 0CSL_D1_V1:R0603_MAN, F.Cu at (105.4, 31.5)
- added R6: 470k, 0CSL_D1_V1:R0603_MAN, F.Cu at (66.4, 56.0)
- added R7: 10k, 0CSL_D1_V1:R0603_MAN, F.Cu at (61.5, 56.5)
- added R8: 210k, 0CSL_D1_V1:R0603_MAN, F.Cu at (109.9, 28.8)
- added U5: TPS63070RNMT, Footprint:QFN50P250X300X100-15N, F.Cu at (57.0, 48.6)
- added U6: ~, Footprint:MSOP-12_MSE, F.Cu at (114.0, 35.0)
- D1, D2, F1, R27, R28: moved to B.Cu
- moved BZ1 154.9 mm to (207.6, 104.5)
- moved C38 118.1 mm to (184.9, 72.0), turned to 90 degrees
- moved R28 111.2 mm to (175.4, 63.5), turned to -90 degrees
- moved C39 108.2 mm to (181.4, 72.0), turned to 90 degrees
- moved R27 108.2 mm to (172.9, 63.5), turned to -90 degrees
- moved F1 108.0 mm to (174.4, 71.5), turned to -90 degrees
- moved J17 107.2 mm to (174.6, 63.4), turned to 180 degrees
- moved D1 103.3 mm to (175.9, 71.5), turned to 90 degrees
- moved U9 101.0 mm to (174.4, 71.5), turned to -90 degrees
- moved D2 99.7 mm to (172.9, 71.5), turned to 90 degrees
- moved U1 99.6 mm to (142.6, 65.1)
- moved C34 66.6 mm to (132.9, 63.1)
- moved C35 66.6 mm to (132.9, 65.6)
- moved C36 66.6 mm to (132.9, 68.1)
- moved D3 5.41 mm to (81.0, 83.0)
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Connections:
- net VDD renamed VDD_MCU
- net VREF renamed VREF+
- D3 pad 1: unconnected-(D3-K-Pad1) -> /ECU_Analog/Pressure Sensor 1
- J17 pad S1: GND -> unconnected-(J17-SHIELD-PadS1)_3
- U2 pad 130: unconnected-(U2-PA11-Pad130) -> FDCAN1_RX
- U2 pad 131: unconnected-(U2-PA12-Pad131) -> FDCAN1_TX
- U2 pad 41: unconnected-(U2-PA0-Pad41) -> /Pressure Sensor 1A
- U2 pad 42: unconnected-(U2-PA1-Pad42) -> /Pressure Sensor 1B
Routing:
- net GND: track 0.00 -> 26.7 mm, vias 0 -> 1
- net /Pressure Sensor 1A: track 0.00 -> 23.9 mm
- net /Pressure Sensor 1B: track 0.00 -> 23.1 mm
- net +5V: track 0.00 -> 14.2 mm
- net /USB_D-: track 0.00 -> 5.70 mm
- net /USB_D+: track 0.00 -> 5.44 mm
- net Net-(J17-CC1): track 0.00 -> 2.87 mm, vias 0 -> 1
- net Net-(J17-CC2): track 0.00 -> 2.72 mm, vias 0 -> 1
- net /D-: track 0.00 -> 1.38 mm, vias 0 -> 1
- net /D+: track 0.00 -> 1.38 mm, vias 0 -> 1
- net (no net): vias 0 -> 50
Other:
- board text added: "Analog"
- board text added: "Digital"
