File: CANopus/CANopus.kicad_sch (KiCad schematic)
At the start: 72 parts, among them J1 Micro_SD_Card_Det1, J17 USB_C_Receptacle_USB2.0_man, J3 JTAG, SW1 SW_Push, U1 SST25VF080B-50-4x-S2Ax, U2 STM32H747IITx, U3 TCAN337G, U9 USBLC6-2SC6, Y1 32.768KHz, Y2 25MHz

Commit message: Pages cleanup
Parts:
- removed C1, C13, C2: 1u, symbol Device:C_Polarized_US
- removed C10, C11, C12, C14, C15, C16, C17, C23, C26, C27, C28, C29, C3, C30, C31, C4, C5, C6, C7, C8, C9: 100n, symbol Device:C
- removed C18: 2.2u ESR < 600m, symbol Device:C
- removed C19: 220p, symbol Device:C
- removed C20, C22: 10u ESR < 20m, symbol Device:C
- removed C21: 4.7u ESR < 100m, symbol Device:C
- removed C33, C40: 2.2u ESR < 100m, symbol Device:C
- removed C41, C42: 4.7u, symbol Device:C
- removed JP1: Jumper_2_Open, symbol Jumper:Jumper_2_Open
- removed JP10, JP11, JP5, JP8, JP9: SMPS, symbol Jumper:SolderJumper_2_Open
- removed JP4, JP6, JP7: LDO, symbol Jumper:SolderJumper_2_Open
- removed L1: 2.2u, symbol Device:L
- removed L2: L_Ferrite, symbol Device:L_Ferrite
- removed U3: TCAN337G, symbol Interface_CAN_LIN:TCAN337G
- added BZ1: Buzzer_TDK_PS1240, 0CSL_D1_V1:Buzzer_TDK_PS1240P02BT_D12.2mmP5mm, symbol 0CSL_D1_V1:Buzzer_TDK_PS1240
Connections:
- net VDD: no longer U2.113 (VDD), U2.126 (VDD), U2.13 (VDD), U2.136 (VDD), U2.152 (VDD), U2.160 (VDD), U2.176 (VDD), U2.25 (VDD), U2.44 (VDD), U2.48 (VDD), U2.65 (VDD), U2.7 (VDD), U2.71 (VDD), U2.84 (VDD), U2.92 (VDD), U2.99 (VDD)
- net VREF: no longer U2.39 (VREF+)
- net FDCAN1_RX: now reaches U2.130 (PA11)
- net FDCAN1_TX: now reaches U2.131 (PA12)
- net VDD55_USB renamed VDD50_USB
- new net VDD_MCU: U2.113 (VDD), U2.126 (VDD), U2.13 (VDD), U2.136 (VDD), U2.152 (VDD), U2.160 (VDD), U2.176 (VDD), U2.25 (VDD), U2.44 (VDD), U2.48 (VDD), U2.65 (VDD), U2.7 (VDD), U2.71 (VDD), U2.84 (VDD), U2.92 (VDD), U2.99 (VDD)
- new net VREF+: U2.39 (VREF+)
- no-connect marks 2 -> 6
Other:
- added sheet ECU_Analog (ECU_ADC.kicad_sch)
- added sheet ECU_Communication (ECU_Communication.kicad_sch)
- added sheet ECU_Decoupling (ECU_Decoupling.kicad_sch)
- added sheet ECU_Power (ECU_Power.kicad_sch)
- note added: "Carte SD"
- note added: "Display Serial Interface"
- note added: "Flash Externe"
- note added: "Switch probablement a retirer"
- note added: "Test point"
- note added: "USB-C"
- note removed: "DSI ?"
- note removed: "REGARDER STARPOINT GROUNDING"
- moved on the sheet: C32, C34, C35, C36, C38, C39, D1, D2, F1, J1, J17, J3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

Commit message: Analog modifs
Signed-off-by: mat7784 <matispoulin@gmail.com>
Connections:
- net Pressure Sensor 1A: now reaches U2.41 (PA0)
- net Pressure Sensor 1B: now reaches U2.42 (PA1)
Other:
- note added: "STM à changer. trop de pins dans pas gros"
Changed lines of the file:
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@@
+		)
+	)
+	(text "STM à changer. trop de pins dans pas gros"
+		(exclude_from_sim no)
+		(at 264.922 165.1 0)
+		(effects
+			(font
+				(size 1.27 1.27)
+			)
 		)
 	)
@@
 	(wire
 		(pts
+			(xy 314.96 105.41) (xy 341.63 105.41)
+		)
+		(stroke
+			(width 0)
+			(type default)
+		)
+	)
+	(wire
+		(pts
 			(xy 524.51 199.39) (xy 520.7 199.39)
 		)
@@
 		(pts
 			(xy 486.41 204.47) (xy 509.27 204.47)
+		)
+		(stroke
+			(width 0)
+			(type default)
+		)
+	)
+	(wire
+		(pts
+			(xy 341.63 102.87) (xy 314.96 102.87)
 		)
 		(stroke
@@
 		)
 	)
+	(label "Pressure Sensor 1A"
+		(at 341.63 102.87 0)
+		(effects
+			(font
+				(size 1.27 1.27)
+			)
+			(justify left bottom)
+		)
+	)
 	(label "LSE1"
 		(at 154.94 153.67 0)
@@
 		(effects
 			(font
+				(size 1.27 1.27)
+			)
+			(justify left bottom)
+		)
+	)
+	(label "Pressure Sensor 1B"
+		(at 341.63 105.41 0)
+		(effects
+			(font

Commit message: Alim
Connections:
- net GND: no longer J17.S1 (SHIELD)
- no-connect marks 6 -> 7
Other:
- moved on the sheet: C32, C38, C39, D1, D2, F1, R27, R28, SW1, U9
